File: 555_badge.kicad_pcb (KiCad board)
At the start: 2 copper layers, 53.8 x 85.6 mm, 15 parts, among them Q1 2N3904, U1 7555

Commit message: Changed R2 to 330k
Parts:
- R2: value 220k -> 330k
Changed lines of the file:
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@@
       (effects (font (size 1 1) (thickness 0.15)))
     )
-    (fp_text value 220k (at 3.81 0 90) (layer F.Fab)
+    (fp_text value 330k (at 3.81 0 90) (layer F.Fab)
       (effects (font (size 1 1) (thickness 0.15)))
     )
