File: Hardware/555_badge.kicad_pcb (KiCad board)
At the start: 2 copper layers, 53.8 x 85.6 mm, 15 parts, among them Q1 2N3904, U1 7555

Commit message: Added some silk. Updated to v02. Panelized design. Created README.
Parts:
- added G***: LOGO, 555_badge:OSHPark-Slide_logo, B.Cu at (153.9, 86.4)
- added G***: LOGO, 555_badge:DigiKey_logo, B.Cu at (167.6, 62.2)
- added G***: LOGO, 555_badge:Maker_io_logo, B.Cu at (141.0, 62.2)
- added G***: LOGO, 555_badge:oshw_logo, B.Cu at (132.3, 121.9)
Other:
- board text added: "-"
- board text added: "Learn how to make this PCB! bit.ly/LearnKiCad"
- board text added: "PCBs by"
- board text added: "v02"
- board text removed: "v00a"

Commit message: Added D1 and D2 refdes to back
Other:
- board text added: "D1"
- board text added: "D2"
Changed lines of the file:
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@@
     (area 126.987299 41.389299 180.860701 127.012701)
     (thickness 1.6)
-    (drawings 20)
+    (drawings 22)
     (tracks 67)
     (zones 0)
@@
     (descr "LED, diameter 3.0mm, 2 pins")
     (tags "LED diameter 3.0mm 2 pins")
-    (fp_text reference D1 (at 1.27 -2.96 90) (layer F.SilkS)
+    (fp_text reference D1 (at 4.572 0 180) (layer F.SilkS)
       (effects (font (size 1 1) (thickness 0.15)))
     )
@@
     (descr "LED, diameter 3.0mm, 2 pins")
     (tags "LED diameter 3.0mm 2 pins")
-    (fp_text reference D2 (at 1.27 -2.96 90) (layer F.SilkS)
+    (fp_text reference D2 (at 4.572 0 180) (layer F.SilkS)
       (effects (font (size 1 1) (thickness 0.15)))
     )
@@
       (xy 0.211682 3.478043) (xy 0.298275 3.47764)) (layer B.SilkS) (width 0.01))
   )
+  (gr_text D2 (at 157.226 73.66) (layer B.SilkS)
+    (effects (font (size 1 1) (thickness 0.1524)) (justify mirror))
+  )
+  (gr_text D1 (at 144.526 73.66) (layer B.SilkS)
+    (effects (font (size 1 1) (thickness 0.1524)) (justify mirror))
+  )
   (gr_text - (at 162.814 75.692) (layer B.SilkS)
